File: pami_2026/_autosave-Power.kicad_sch (KiCad schematic)
At the start: 37 parts, among them Q1 PMOS, Q2 PMOS, U2 AP63205WU, U3 DRV8871DDA, U5 AP63203WU, U6 DRV8871DDA

Commit message: fix
Parts:
- renumbered BAU to BAU1, C_BATT to C_BATT1
Changed lines of the file:
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@@
 		(dnp no)
 		(fields_autoplaced yes)
-		(property "Reference" "C_BATT"
+		(property "Reference" "C_BATT1"
 			(at 139.065 21.59 0)
 			(effects
@@
 			(project ""
 				(path "/2e16a05b-e8ca-4fff-9c3e-5c880745daa6/ed527990-c321-4ebf-9ae6-9a3c892317c7"
-					(reference "C_BATT")
+					(reference "C_BATT1")
 					(unit 1)
 				)
@@
 		(dnp no)
 		(fields_autoplaced yes)
-		(property "Reference" "BAU"
+		(property "Reference" "BAU1"
 			(at 158.75 20.9549 90)
 			(effects
@@
 			(project "pami_2026"
 				(path "/2e16a05b-e8ca-4fff-9c3e-5c880745daa6/ed527990-c321-4ebf-9ae6-9a3c892317c7"
-					(reference "BAU")
-					(unit 1)
-				)
+					(reference "BAU1")
+					(unit 1)
+				)
