File: pami_2026/asu.kicad_sch (KiCad schematic)
At the start: 23 parts, among them J10 Conn_01x02_Pin, J2 Conn_01x03_Pin, J3 Conn_01x03_Pin, J4 Conn_01x03_Pin, J5 Conn_01x06, J6 Conn_01x06, J7 Conn_01x04_Pin, J8 Conn_01x04_Pin, SW1 SW_Reed

Commit message: Feat: BOM LCSC + big plan de masse
Parts:
- D2, D3, D4, D6: LCSC (none) -> C965799
- J10, SW1: LCSC (none) -> C32713268
- J2, J3, J4: LCSC (none) -> C32713269
- J5, J6: LCSC (none) -> C37208
- J7, J8: LCSC (none) -> C42431808
- R2: LCSC (none) -> C4045076
- R21, R3: LCSC (none) -> C22548
- R4: LCSC (none) -> C114662
- SWPushBoot1, SWPushReset1: LCSC (none) -> C967701
Changed lines of the file:
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@@
 			)
 		)
+		(property "LCSC" "C22548"
+			(at 105.41 97.79 0)
+			(effects
+				(font
+					(size 1.27 1.27)
+				)
+				(hide yes)
+			)
+		)
 		(pin "1"
 		)
@@
 			)
 		)
+		(property "LCSC" "C965799"
+			(at 85.09 105.41 90)
+			(effects
+				(font
+					(size 1.27 1.27)
+				)
+				(hide yes)
+			)
+		)
 		(pin "2"
 		)
@@
 			)
 		)
+		(property "LCSC" "C967701"
+			(at 99.06 55.88 0)
+			(effects
+				(font
+					(size 1.27 1.27)
+				)
+				(hide yes)
+			)
+		)
 		(pin "2"
 		)
@@
 			)
 		)
+		(property "LCSC" "C37208"
+			(at 148.59 26.67 0)
+			(effects
+				(font
+					(size 1.27 1.27)
+				)
+				(hide yes)
+			)
+		)
 		(pin "6"
 		)
@@
 			)
 		)
+		(property "LCSC" ""
+			(at 85.09 93.98 90)
+			(effects
+				(font
+					(size 1.27 1.27)
+				)
+				(hide yes)
+			)
+		)
 		(pin "1"
 		)
@@
 			)
 		)
+		(property "LCSC" "C965799"
+			(at 95.25 105.41 90)
+			(effects
+				(font
+					(size 1.27 1.27)
+				)
+				(hide yes)
+			)
+		)
 		(pin "2"
 		)
@@
 			)
 		)
+		(property "LCSC" ""
+			(at 105.41 93.98 90)
+			(effects
+				(font
+					(size 1.27 1.27)
+				)
+				(hide yes)
+			)
+		)
 		(pin "1"
 		)
@@
 			)
 		)
+		(property "LCSC" "C32713268"
+			(at 76.2 31.75 90)
+			(effects
+				(font
+					(size 1.27 1.27)
+				)
+				(hide yes)
+			)
+		)
 		(pin "1"
 		)
@@
 			)
 		)
+		(property "LCSC" ""
+			(at 95.25 93.98 90)
+			(effects
+				(font
+					(size 1.27 1.27)
+				)
+				(hide yes)
+			)
+		)
 		(pin "1"
 		)
@@
 			)
 		)
+		(property "LCSC" "C37208"
+			(at 118.11 26.67 0)
+			(effects
+				(font
+					(size 1.27 1.27)
+				)
+				(hide yes)
+			)
+		)
 		(pin "6"
 		)
@@
 			)
 		)
+		(property "LCSC" "C965799"
+			(at 105.41 105.41 90)
+			(effects
+				(font
+					(size 1.27 1.27)
+				)
+				(hide yes)
+			)
+		)
 		(pin "2"
 		)
@@
 			)
 		)
+		(property "LCSC" "C42431808"
+			(at 33.02 29.21 0)
+			(effects
+				(font
+					(size 1.27 1.27)
+				)
+				(hide yes)
+			)
+		)
 		(pin "2"
 		)
@@
 			)
 		)
+		(property "LCSC" "C22548"
+			(at 85.09 97.79 0)
+			(effects
+				(font
+					(size 1.27 1.27)
+				)
+				(hide yes)
+			)
+		)
 		(pin "1"
 		)
@@
 			)
 		)
+		(property "LCSC" ""
+			(at 73.66 93.98 90)
+			(effects
+				(font
+					(size 1.27 1.27)
+				)
+				(hide yes)
+			)
+		)
 		(pin "1"
 		)
@@
 			)
 		)
+		(property "LCSC" "C32713269"
+			(at 35.56 106.68 0)
+			(effects
+				(font
+					(size 1.27 1.27)
+				)
+				(hide yes)
+			)
+		)
 		(pin "1"
 		)
@@
 			)
 		)
+		(property "LCSC" "C32713269"
+			(at 35.56 90.17 0)
+			(effects
+				(font
+					(size 1.27 1.27)
+				)
+				(hide yes)
+			)
+		)
 		(pin "1"
 		)
@@
 			)
 		)
+		(property "LCSC" "C4045076"
+			(at 73.66 97.79 0)
+			(effects
+				(font
+					(size 1.27 1.27)
+				)
+				(hide yes)
+			)
+		)
 		(pin "1"
 		)
@@
 			)
 		)
+		(property "LCSC" "C32713268"
+			(at 76.2 25.4 0)
+			(effects
+				(font
+					(size 1.27 1.27)
+				)
+				(hide yes)
+			)
+		)
 		(pin "2"
 		)
@@
 			)
 		)
+		(property "LCSC" "C114662"
+			(at 95.25 97.79 0)
+			(effects
+				(font
+					(size 1.27 1.27)
+				)
+				(hide yes)
+			)
+		)
 		(pin "1"
 		)
@@
 			)
 		)
+		(property "LCSC" "C42431808"
+			(at 67.31 57.15 0)
+			(effects
+				(font
+					(size 1.27 1.27)
+				)
+				(hide yes)
+			)
+		)
 		(pin "4"
 		)
@@
 			)
 		)
+		(property "LCSC" "C32713269"
+			(at 29.21 66.04 90)
+			(effects
+				(font
+					(size 1.27 1.27)
+				)
+				(hide yes)
+			)
+		)
 		(pin "3"
 		)
@@
 			)
 		)
+		(property "LCSC" "C967701"
+			(at 99.06 67.31 0)
+			(effects
+				(font
+					(size 1.27 1.27)
+				)
+				(hide yes)
+			)
+		)
 		(pin "2"
 		)
@@
 			(effects
 				(font
+					(size 1.27 1.27)
+				)
+				(hide yes)
+			)
+		)
+		(property "LCSC" "C965799"
+			(at 73.66 105.41 90)
+			(effects
+				(font

Commit message: fix
Parts:
- TP1, TP2, TP3, TP4: now left out of the parts list
- renumbered J5 to DC_A, J6 to DC_B, J3 to SERVO_1, J4 to SERVO_2, J10 to SW_TEAM, D2 to S_3.3V, D3 to S_5V, D4 to S_BATT, D6 to S_ESP, J2 to TEAM_RGB, J7 to UART, J8 to US
Changed lines of the file:
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@@
 		(exclude_from_sim no)
 		(at 93.98 15.24 0)
-		(size 64.77 26.67)
+		(size 71.12 26.67)
 		(margins 0.9525 0.9525 0.9525 0.9525)
 		(stroke
@@
 		(dnp no)
 		(fields_autoplaced yes)
-		(property "Reference" "D3"
+		(property "Reference" "S_5V"
 			(at 88.9 105.7274 90)
 			(effects
@@
 			(project "pami_2026"
 				(path "/2e16a05b-e8ca-4fff-9c3e-5c880745daa6/bb7fbca0-80fe-418e-a09d-cb4c86ee0cfe"
-					(reference "D3")
+					(reference "S_5V")
 					(unit 1)
 				)
@@
 		(dnp no)
 		(fields_autoplaced yes)
-		(property "Reference" "J6"
-			(at 148.59 40.64 0)
+		(property "Reference" "DC_B"
+			(at 151.13 26.6699 0)
 			(effects
 				(font
 					(size 1.27 1.27)
 				)
+				(justify left)
 			)
 		)
 		(property "Value" "Conn_01x06"
-			(at 148.59 38.1 0)
+			(at 151.13 29.2099 0)
 			(effects
 				(font
 					(size 1.27 1.27)
 				)
+				(justify left)
 			)
 		)
@@
 			(project "pami_2026"
 				(path "/2e16a05b-e8ca-4fff-9c3e-5c880745daa6/bb7fbca0-80fe-418e-a09d-cb4c86ee0cfe"
-					(reference "J6")
+					(reference "DC_B")
 					(unit 1)
 				)
@@
 		(unit 1)
 		(exclude_from_sim no)
-		(in_bom yes)
+		(in_bom no)
 		(on_board yes)
 		(dnp no)
@@
 		(dnp no)
 		(fields_autoplaced yes)
-		(property "Reference" "D4"
+		(property "Reference" "S_BATT"
 			(at 99.06 105.7274 90)
 			(effects
@@
 			(project "pami_2026"
 				(path "/2e16a05b-e8ca-4fff-9c3e-5c880745daa6/bb7fbca0-80fe-418e-a09d-cb4c86ee0cfe"
-					(reference "D4")
+					(reference "S_BATT")
 					(unit 1)
 				)
@@
 		(unit 1)
 		(exclude_from_sim no)
-		(in_bom yes)
+		(in_bom no)
 		(on_board yes)
 		(dnp no)
@@
 		(dnp no)
 		(fields_autoplaced yes)
-		(property "Reference" "J10"
+		(property "Reference" "SW_TEAM"
 			(at 77.47 31.1149 90)
 			(effects
@@
 			(project "pami_2026"
 				(path "/2e16a05b-e8ca-4fff-9c3e-5c880745daa6/bb7fbca0-80fe-418e-a09d-cb4c86ee0cfe"
-					(reference "J10")
+					(reference "SW_TEAM")
 					(unit 1)
 				)
@@
 		(unit 1)
 		(exclude_from_sim no)
-		(in_bom yes)
+		(in_bom no)
 		(on_board yes)
 		(dnp no)
@@
 		(dnp no)
 		(fields_autoplaced yes)
-		(property "Reference" "J5"
-			(at 118.11 40.64 0)
+		(property "Reference" "DC_A"
+			(at 120.65 26.6699 0)
 			(effects
 				(font
 					(size 1.27 1.27)
 				)
+				(justify left)
 			)
 		)
 		(property "Value" "Conn_01x06"
-			(at 118.11 38.1 0)
+			(at 120.65 29.2099 0)
 			(effects
 				(font
 					(size 1.27 1.27)
 				)
+				(justify left)
 			)
 		)
@@
 			(project ""
 				(path "/2e16a05b-e8ca-4fff-9c3e-5c880745daa6/bb7fbca0-80fe-418e-a09d-cb4c86ee0cfe"
-					(reference "J5")
+					(reference "DC_A")
 					(unit 1)
 				)
@@
 		(dnp no)
 		(fields_autoplaced yes)
-		(property "Reference" "D6"
+		(property "Reference" "S_ESP"
 			(at 109.22 105.7274 90)
 			(effects
@@
 			(project "pami_2026"
 				(path "/2e16a05b-e8ca-4fff-9c3e-5c880745daa6/bb7fbca0-80fe-418e-a09d-cb4c86ee0cfe"
-					(reference "D6")
+					(reference "S_ESP")
 					(unit 1)
 				)
@@
 		(dnp no)
 		(fields_autoplaced yes)
-		(property "Reference" "J8"
+		(property "Reference" "US"
 			(at 34.29 26.6699 0)
 			(effects
@@
 			(project ""
 				(path "/2e16a05b-e8ca-4fff-9c3e-5c880745daa6/bb7fbca0-80fe-418e-a09d-cb4c86ee0cfe"
-					(reference "J8")
+					(reference "US")
 					(unit 1)
 				)
@@
 		(unit 1)
 		(exclude_from_sim no)
-		(in_bom yes)
+		(in_bom no)
 		(on_board yes)
 		(dnp no)
@@
 		(dnp no)
 		(fields_autoplaced yes)
-		(property "Reference" "J4"
+		(property "Reference" "SERVO_2"
 			(at 36.83 105.4099 0)
 			(effects
@@
 			(project "pami_2026"
 				(path "/2e16a05b-e8ca-4fff-9c3e-5c880745daa6/bb7fbca0-80fe-418e-a09d-cb4c86ee0cfe"
-					(reference "J4")
+					(reference "SERVO_2")
 					(unit 1)
 				)
@@
 		(dnp no)
 		(fields_autoplaced yes)
-		(property "Reference" "J3"
+		(property "Reference" "SERVO_1"
 			(at 36.83 88.8999 0)
 			(effects
@@
 			(project ""
 				(path "/2e16a05b-e8ca-4fff-9c3e-5c880745daa6/bb7fbca0-80fe-418e-a09d-cb4c86ee0cfe"
-					(reference "J3")
+					(reference "SERVO_1")
 					(unit 1)
 				)
@@
 		(dnp no)
 		(fields_autoplaced yes)
-		(property "Reference" "J7"
+		(property "Reference" "UART"
 			(at 68.58 54.6099 0)
 			(effects
@@
 			(project ""
 				(path "/2e16a05b-e8ca-4fff-9c3e-5c880745daa6/bb7fbca0-80fe-418e-a09d-cb4c86ee0cfe"
-					(reference "J7")
+					(reference "UART")
 					(unit 1)
 				)
@@
 		(dnp no)
 		(fields_autoplaced yes)
-		(property "Reference" "J2"
+		(property "Reference" "TEAM_RGB"
 			(at 29.21 68.58 90)
 			(effects
@@
 			(project ""
 				(path "/2e16a05b-e8ca-4fff-9c3e-5c880745daa6/bb7fbca0-80fe-418e-a09d-cb4c86ee0cfe"
-					(reference "J2")
+					(reference "TEAM_RGB")
 					(unit 1)
 				)
@@
 		(dnp no)
 		(fields_autoplaced yes)
-		(property "Reference" "D2"
+		(property "Reference" "S_3.3V"
 			(at 77.47 105.7274 90)
 			(effects
@@
 			(project ""
 				(path "/2e16a05b-e8ca-4fff-9c3e-5c880745daa6/bb7fbca0-80fe-418e-a09d-cb4c86ee0cfe"
-					(reference "D2")
+					(reference "S_3.3V")
 					(unit 1)
 				)

Commit message: Cleanup
Parts:
- removed SERVO_1, SERVO_2, TEAM_RGB: Conn_01x03_Pin, Connector_PinHeader_2.54mm:PinHeader_1x03_P2.54mm_Vertical, symbol Connector:Conn_01x03_Pin
- removed SW1: SW_Reed, Connector_PinHeader_2.54mm:PinHeader_1x02_P2.54mm_Vertical, symbol Switch:SW_Reed
- removed SWPushBoot1, SWPushReset1: SMD_6.2x6.2mm_h7.0mm, PCM_SparkFun-Switch:Push_SMD_6.2x6.2mm, symbol PCM_SparkFun-Switch:SPST_Push_SMD_6.2x6.2mm_h7.0mm
- removed SW_TEAM: Conn_01x02_Pin, Connector_PinHeader_2.54mm:PinHeader_1x02_P2.54mm_Vertical, symbol Connector:Conn_01x02_Pin
- removed UART, US: Conn_01x04_Pin, Connector_PinHeader_2.54mm:PinHeader_1x04_P2.54mm_Vertical, symbol Connector:Conn_01x04_Pin
- added C13, C15: 47uF, PCM_SparkFun-Capacitor:Panasonic_F, symbol Device:C_Polarized
- added C14, C16: 100nF, Capacitor_SMD:C_0603_1608Metric, symbol Device:C
- added R14, R19: 24K, Resistor_SMD:R_0603_1608Metric, symbol Device:R
- added R15, R16, R17, R18: 10K, Resistor_SMD:R_0603_1608Metric, symbol Device:R
- added U3, U6: DRV8871DDA, Package_SO:Texas_HTSOP-8-1EP_3.9x4.9mm_P1.27mm_EP2.95x4.9mm_Mask2.4x3.1mm_ThermalVias, symbol Driver_Motor:DRV8871DDA
Connections:
- net BATT: now also C13.1, C14.1, C15.1, C16.1, U3.5 (VM), U6.5 (VM)
- net DC_OUT_A+: now also U3.6 (OUT1)
- net DC_OUT_A-: now also U3.8 (OUT2)
- net DC_OUT_B+: now also U6.6 (OUT1)
- net DC_OUT_B-: now also U6.8 (OUT2)
- net GND: now also C13.2, C14.2, C15.2, C16.2, R14.1, R15.2, R16.2, R17.2, R18.2, R19.1, U3.1 (GND), U3.7 (GND), U3.9 (GND), U6.1 (GND), U6.7 (GND), U6.9 (GND)
- new net: R19.2, U3.4 (ILIM)
- new net: R14.2, U6.4 (ILIM)
- new net DC_A1: R18.1, U3.3 (IN1)
- new net DC_A2: R17.1, U3.2 (IN2)
- new net DC_B1: R16.1, U6.3 (IN1)
- new net DC_B2: R15.1, U6.2 (IN2)
Other:
- moved on the sheet: DC_A, DC_B, R2, R21, R3, R4, S_3.3V, S_5V, S_BATT, S_ESP, TP1, TP2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
