File: pami_2026/asu.kicad_sch (KiCad schematic)
At the start: 26 parts, among them U3 DRV8871DDA, U6 DRV8871DDA

Commit message: Fixes and updates to v2
Parts:
- renumbered DC_A to DC_A1, DC_B to DC_B1, S_3.3V to S_3.3V1, S_5V to S_5V2, S_BATT to S_BATT1, S_ESP to S_ESP1
Changed lines of the file:
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@@
 		(dnp no)
 		(fields_autoplaced yes)
-		(property "Reference" "S_5V"
+		(property "Reference" "S_5V2"
 			(at 78.74 101.9174 90)
 			(effects
@@
 			(project "pami_2026"
 				(path "/2e16a05b-e8ca-4fff-9c3e-5c880745daa6/bb7fbca0-80fe-418e-a09d-cb4c86ee0cfe"
-					(reference "S_5V")
+					(reference "S_5V2")
 					(unit 1)
 				)
@@
 		(dnp no)
 		(fields_autoplaced yes)
-		(property "Reference" "DC_B"
+		(property "Reference" "DC_B1"
 			(at 203.2 130.8099 0)
 			(effects
@@
 			(project "pami_2026"
 				(path "/2e16a05b-e8ca-4fff-9c3e-5c880745daa6/bb7fbca0-80fe-418e-a09d-cb4c86ee0cfe"
-					(reference "DC_B")
+					(reference "DC_B1")
 					(unit 1)
 				)
@@
 		(dnp no)
 		(fields_autoplaced yes)
-		(property "Reference" "S_BATT"
+		(property "Reference" "S_BATT1"
 			(at 88.9 101.9174 90)
 			(effects
@@
 			(project "pami_2026"
 				(path "/2e16a05b-e8ca-4fff-9c3e-5c880745daa6/bb7fbca0-80fe-418e-a09d-cb4c86ee0cfe"
-					(reference "S_BATT")
+					(reference "S_BATT1")
 					(unit 1)
 				)
@@
 		(dnp no)
 		(fields_autoplaced yes)
-		(property "Reference" "DC_A"
+		(property "Reference" "DC_A1"
 			(at 172.72 130.8099 0)
 			(effects
@@
 			(project "pami_2026"
 				(path "/2e16a05b-e8ca-4fff-9c3e-5c880745daa6/bb7fbca0-80fe-418e-a09d-cb4c86ee0cfe"
-					(reference "DC_A")
+					(reference "DC_A1")
 					(unit 1)
 				)
@@
 		(dnp no)
 		(fields_autoplaced yes)
-		(property "Reference" "S_ESP"
+		(property "Reference" "S_ESP1"
 			(at 99.06 101.9174 90)
 			(effects
@@
 			(project "pami_2026"
 				(path "/2e16a05b-e8ca-4fff-9c3e-5c880745daa6/bb7fbca0-80fe-418e-a09d-cb4c86ee0cfe"
-					(reference "S_ESP")
+					(reference "S_ESP1")
 					(unit 1)
 				)
@@
 		(dnp no)
 		(fields_autoplaced yes)
-		(property "Reference" "S_3.3V"
+		(property "Reference" "S_3.3V1"
 			(at 67.31 101.9174 90)
 			(effects
@@
 			(project "pami_2026"
 				(path "/2e16a05b-e8ca-4fff-9c3e-5c880745daa6/bb7fbca0-80fe-418e-a09d-cb4c86ee0cfe"
-					(reference "S_3.3V")
+					(reference "S_3.3V1")
 					(unit 1)
 				)
